File: flashlight.kicad_pcb (KiCad board)
At the start: 2 copper layers, 45 x 120 mm, 39 parts, among them J1 USB_B_Micro, Q1 HSS2333, Q2 HSS2333, SW1 SW_DIP_x01, U1 LP4054HB5F, U2 MT3608

Commit message: v0.1
Parts:
- added C1: 4u7/10V, Capacitor_SMD:C_0603_1608Metric, B.Cu at (102.1, 51.8)
- added C2: 4u7/10V, Capacitor_SMD:C_0603_1608Metric, B.Cu at (94.0, 54.4)
- added R1: 2k2, Resistor_SMD:R_0603_1608Metric, B.Cu at (112.3, 45.7)
- moved R3 12.3 mm to (84.8, 55.9), turned to 180 degrees
- moved R2 4.67 mm to (93.0, 43.2), turned to 90 degrees
- moved R4 3.87 mm to (100.1, 45.2), turned to 90 degrees
- moved D3 3.42 mm to (88.9, 52.3)
- moved D2 3.37 mm to (89.2, 45.2), turned to 0 degrees
- moved Q1 1.37 mm to (89.3, 58.8)
Connections:
- R3 pad 1: Net-(D3-K) -> GND
- R3 pad 2: GND -> Net-(D3-K)
Routing:
- net Net-(D3-A): track 9.65 -> 57.5 mm
- net Net-(U1-PROG): track 0.00 -> 4.63 mm
- net Net-(D1-K): track 40.2 -> 35.9 mm
- net Net-(D2-K): track 3.08 -> 6.00 mm
- net Net-(D3-K): track 5.12 -> 6.52 mm
- net Net-(Q1-D): track 29.2 -> 30.6 mm
- net Net-(BT1-+): track 9.29 -> 7.93 mm

Commit message: v0.2
Parts:
- moved R3 16.1 mm to (94.6, 43.0)
- moved D4 11.1 mm to (91.5, 59.3), turned to 180 degrees
- moved C1 9.04 mm to (93.1, 51.7), turned to -90 degrees
- moved D3 8.87 mm to (90.0, 43.5), turned to 180 degrees
- moved R1 8.73 mm to (103.7, 47.6)
- moved R4 7.84 mm to (95.6, 51.7), turned to -90 degrees
- moved U1 7.56 mm to (99.7, 48.1)
- moved Q2 7.23 mm to (99.6, 56.2)
- moved R2 4.55 mm to (94.1, 47.6)
- moved Q1 4.20 mm to (92.1, 55.6)
- moved D1 2.07 mm to (90.0, 50.6)
- moved D2 2.05 mm to (90.0, 47.1), turned to 180 degrees
- moved C2 1.97 mm to (95.6, 55.5), turned to -90 degrees
Routing:
- net Net-(D3-A): track 57.5 -> 33.6 mm
- net Net-(Q1-D): track 30.6 -> 17.7 mm
- net Net-(D1-K): track 35.9 -> 31.2 mm
- net Net-(D3-K): track 6.52 -> 2.98 mm
- net Net-(D4-K): track 28.4 -> 31.0 mm
- net Net-(BT1-+): track 7.93 -> 10.5 mm
- net Net-(D2-K): track 6.00 -> 4.21 mm
- net Net-(U1-PROG): track 4.63 -> 3.19 mm

Commit message: v0.3
Parts:
- moved R3 16.1 mm to (84.8, 55.9)
- moved D4 11.1 mm to (102.6, 59.4), turned to 90 degrees
- moved C1 9.04 mm to (102.1, 51.8), turned to 180 degrees
- moved D3 8.87 mm to (88.9, 52.3), turned to 90 degrees
- moved R4 7.84 mm to (100.1, 45.2), turned to 90 degrees
- moved U1 7.56 mm to (107.2, 47.2)
- moved Q2 7.23 mm to (106.2, 53.3)
- moved R1 7.11 mm to (110.2, 44.7), turned to 90 degrees
- moved R2 4.55 mm to (93.0, 43.2)
- moved Q1 4.20 mm to (89.3, 58.8)
- moved D1 2.07 mm to (90.6, 48.6)
- moved D2 2.05 mm to (89.2, 45.2), turned to 0 degrees
- moved C2 1.97 mm to (94.0, 54.4), turned to 180 degrees
Routing:
- net Net-(D3-A): track 33.6 -> 49.1 mm
- net Net-(Q1-D): track 17.7 -> 30.6 mm
- net Net-(D1-K): track 31.2 -> 35.9 mm
- net Net-(D3-K): track 2.98 -> 6.52 mm
- net Net-(D4-K): track 31.0 -> 28.4 mm
- net Net-(BT1-+): track 10.5 -> 7.93 mm
- net Net-(D2-K): track 4.21 -> 6.00 mm
- net Net-(U1-PROG): track 3.19 -> 2.34 mm

Commit message: v0.4_work
Parts:
- moved R3 9.77 mm to (93.7, 51.8), turned to 90 degrees
- moved C1 9.09 mm to (94.0, 47.8), turned to 90 degrees
- moved U1 6.43 mm to (101.1, 45.2)
- moved D4 6.27 mm to (97.3, 56.1)
- moved Q2 5.81 mm to (100.5, 52.2)
- moved R4 5.68 mm to (96.4, 49.5), turned to -90 degrees
- moved R1 5.60 mm to (104.6, 45.0), turned to -90 degrees
- moved Q1 3.65 mm to (90.2, 55.3)
- moved C2 1.80 mm to (94.2, 56.1), turned to -90 degrees
- moved D3 1.65 mm to (90.2, 51.3), turned to 180 degrees
- moved R2 1.02 mm to (91.9, 43.2)
- moved D2 0.56 mm to (89.4, 44.7), turned to -90 degrees
Routing:
- net Net-(Q1-D): track 30.6 -> 19.9 mm
- net Net-(D1-K): track 35.9 -> 25.8 mm
- net Net-(D3-A): track 49.1 -> 42.8 mm
- net Net-(D3-K): track 6.52 -> 2.95 mm
- net Net-(D2-K): track 6.00 -> 2.65 mm
- net Net-(BT1-+): track 7.93 -> 11.1 mm
- net Net-(D4-K): track 28.4 -> 29.7 mm

Commit message: jlcpcb completed
Parts:
- R10, R8, R9: moved to B.Cu
- moved D15 119.2 mm to (97.1, 43.6)
- moved R9 117.1 mm to (94.5, 43.4), turned to -90 degrees
- moved D14 108.6 mm to (99.9, 51.0), turned to 180 degrees
- moved D13 101.0 mm to (97.1, 58.4)
- moved D20 91.5 mm to (97.1, 80.7)
- moved D12 90.7 mm to (99.9, 65.9), turned to 180 degrees
- moved D11 84.1 mm to (97.1, 73.3)
- moved D19 81.9 mm to (99.9, 88.2), turned to 180 degrees
- moved D18 77.0 mm to (97.1, 95.6)
- moved D17 68.5 mm to (99.9, 103.0), turned to 180 degrees
- moved D16 66.0 mm to (97.1, 110.4)
- moved R10 65.4 mm to (104.9, 98.5), turned to -90 degrees
- moved D10 58.0 mm to (97.1, 117.8)
- moved D9 50.4 mm to (99.9, 125.3), turned to 180 degrees
- moved R8 50.0 mm to (104.8, 111.5), turned to 90 degrees
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Routing:
- net VDD: track 0.00 -> 110.9 mm, vias 0 -> 3
- net Net-(D20-K): track 0.00 -> 22.8 mm, vias 0 -> 1
- net Net-(U2-IN): track 0.00 -> 22.5 mm
- net Net-(D10-K): track 0.00 -> 10.1 mm, vias 0 -> 1
- net Net-(D7-K): track 0.00 -> 7.63 mm
- net Net-(D17-K): track 0.00 -> 7.63 mm
- net Net-(D19-K): track 0.00 -> 7.48 mm
- net Net-(D10-A): track 0.00 -> 7.48 mm
- net Net-(D14-K): track 0.00 -> 7.48 mm
- net Net-(D12-K): track 0.00 -> 7.48 mm
- net Net-(D6-K): track 0.00 -> 7.44 mm
- net Net-(D11-K): track 0.00 -> 7.44 mm
- net Net-(D13-K): track 0.00 -> 7.44 mm
- net Net-(D18-K): track 0.00 -> 7.44 mm
- net Net-(D8-K): track 0.00 -> 7.34 mm
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- removed copper zone on F.Cu, net GND
Other:
- outline, holes or cut-outs redrawn
