File: flashlight.kicad_sch (KiCad schematic)
At the start: 25 parts, among them J1 USB_B_Micro, J2 Conn_01x03_Pin, Q1 HSS2333, Q2 HSS2333, SW1 SW_DIP_x01, U1 LP4054HB5F, U2 MT3608

Commit message: v2.2.2
Parts:
- BT1, L1: now left out of the parts list
- D2: value RED -> CHARGING; Color (none) -> Red
- D3: value GREEN -> CHARGED; Color (none) -> Green
- Q1, Q2: LCSC C845590 -> C15127
Connections:
- net +5V: no longer names the net of D1.2 (A), J1.1 (VBUS)
Other:
- note added: "12.6V"
Changed lines of the file:
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@@
   (junction (at 241.3 58.42) (diameter 0) (color 0 0 0 0)
-  )
-  (junction (at 38.1 58.42) (diameter 0) (color 0 0 0 0)
   )
   (junction (at 259.08 77.47) (diameter 0) (color 0 0 0 0)
@@
     (stroke (width 0) (type default))
   )
-  (wire (pts (xy 38.1 58.42) (xy 35.56 58.42))
-    (stroke (width 0) (type default))
-  )
   (wire (pts (xy 144.78 58.42) (xy 153.67 58.42))
     (stroke (width 0) (type default))
@@
     (stroke (width 0) (type default))
   )
-  (wire (pts (xy 38.1 48.26) (xy 38.1 58.42))
-    (stroke (width 0) (type default))
-  )
   (wire (pts (xy 129.54 156.21) (xy 129.54 158.75))
     (stroke (width 0) (type default))
@@
     (stroke (width 0) (type default))
   )
-  (wire (pts (xy 38.1 58.42) (xy 41.91 58.42))
-    (stroke (width 0) (type default))
-  )
   (wire (pts (xy 93.98 116.84) (xy 93.98 113.03))
     (stroke (width 0) (type default))
@@
     (stroke (width 0) (type default))
   )
+  (wire (pts (xy 35.56 58.42) (xy 41.91 58.42))
+    (stroke (width 0) (type default))
+  )
   (wire (pts (xy 68.58 58.42) (xy 68.58 66.04))
     (stroke (width 0) (type default))
@@
   (wire (pts (xy 229.87 90.17) (xy 229.87 82.55))
     (stroke (width 0) (type default))
+  )
+  (text "12.6V" (at 261.62 57.785 0)
+    (effects (font (size 1.27 1.27)) (justify left bottom))
   )
   (text "4u7/10V" (at 57.15 74.93 0)
@@
   )
   (label "Vf=0.6V" (at 237.49 77.47 0) (fields_autoplaced)
-    (effects (font (size 1.27 1.27)) (justify left bottom))
-  )
-  (label "12.6V" (at 261.62 58.42 0) (fields_autoplaced)
     (effects (font (size 1.27 1.27)) (justify left bottom))
   )
@@
     )
   )
-  (symbol (lib_id "power:+5V") (at 38.1 48.26 0) (unit 1)
-    (in_bom yes) (on_board yes) (dnp no) (fields_autoplaced)
-    (property "Reference" "#PWR02" (at 38.1 52.07 0)
-      (effects (font (size 1.27 1.27)) hide)
-    )
-    (property "Value" "+5V" (at 40.64 46.99 0)
-      (effects (font (size 1.27 1.27)) (justify left))
-    )
-    (property "Footprint" "" (at 38.1 48.26 0)
-      (effects (font (size 1.27 1.27)) hide)
-    )
-    (property "Datasheet" "" (at 38.1 48.26 0)
-      (effects (font (size 1.27 1.27)) hide)
-    )
-    (pin "1")
-    (instances
-      (project "flashlight"
-        (path "/98487160-c149-430f-8381-4af03ebcbf31"
-          (reference "#PWR02") (unit 1)
-        )
-      )
-    )
-  )
   (symbol (lib_id "Connector:Conn_01x03_Pin") (at 119.38 153.67 0) (unit 1)
     (in_bom no) (on_board yes) (dnp no) (fields_autoplaced)
@@
   )
   (symbol (lib_id "Device:Battery_Cell") (at 166.37 91.44 0) (unit 1)
-    (in_bom yes) (on_board yes) (dnp no) (fields_autoplaced)
+    (in_bom no) (on_board yes) (dnp no) (fields_autoplaced)
     (property "Reference" "BT1" (at 170.18 88.3285 0)
       (effects (font (size 1.27 1.27)) (justify left))
@@
       (effects (font (size 1.27 1.27)) (justify right))
     )
-    (property "Value" "RED" (at 72.39 72.7075 90)
+    (property "Value" "CHARGING" (at 72.39 72.7075 90)
       (effects (font (size 1.27 1.27)) (justify right))
     )
@@
     )
     (property "LCSC" "C2286" (at 68.58 69.85 90)
+      (effects (font (size 1.27 1.27)) hide)
+    )
+    (property "Color" "Red" (at 68.58 69.85 90)
       (effects (font (size 1.27 1.27)) hide)
     )
@@
   )
   (symbol (lib_id "Device:L") (at 229.87 58.42 90) (unit 1)
-    (in_bom yes) (on_board yes) (dnp no) (fields_autoplaced)
+    (in_bom no) (on_board yes) (dnp no) (fields_autoplaced)
     (property "Reference" "L1" (at 229.87 53.34 90)
       (effects (font (size 1.27 1.27)))
@@
       (effects (font (size 1.27 1.27)) (justify right))
     )
-    (property "Value" "GREEN" (at 72.39 109.5375 90)
+    (property "Value" "CHARGED" (at 72.39 109.5375 90)
       (effects (font (size 1.27 1.27)) (justify right))
     )
@@
     )
     (property "LCSC" "C2297" (at 68.58 106.68 90)
+      (effects (font (size 1.27 1.27)) hide)
+    )
+    (property "Color" "Green" (at 68.58 106.68 90)
       (effects (font (size 1.27 1.27)) hide)
     )
@@
       (effects (font (size 1.27 1.27)) (justify left) hide)
     )
-    (property "LCSC" "C845590" (at 144.78 49.53 90)
+    (property "LCSC" "C15127" (at 144.78 49.53 90)
       (effects (font (size 1.27 1.27)) hide)
     )
@@
       (effects (font (size 1.27 1.27)) (justify left) hide)
     )
-    (property "LCSC" "C845590" (at 152.4 87.63 90)
-      (effects (font (size 1.27 1.27)) hide)
-    )
+    (property "LCSC" "C15127" (at 152.4 87.63 90)
+      (effects (font (size 1.27 1.27)) hide)
+    )
