File: flashlight.kicad_sch (KiCad schematic)
At the start: 23 parts, among them J1 USB_B_Micro, J2 Conn_01x03_Pin, Q2 HSS2333, SW1 SW_DIP_x01, U1 XB4908A, U2 MT3608, U3 TP4057, U4 R6BHC-A05_LED-19-223

Commit message: xb4908 v2.5
Parts:
- U2: footprint Package_TO_SOT_SMD:SOT-23-6 -> SparkFun-Semiconductor-Standard:SOT23-6-Tight
Connections:
- net GND: no longer C3.2, C4.2, J2.2 (Pin_2), J2.3 (Pin_3), R6.1, U1.3 (VM), U1.4 (VM), U2.2 (GND)
- new net Earth_Protective: C3.2, C4.2, J2.2 (Pin_2), J2.3 (Pin_3), R6.1, U1.3 (VM), U1.4 (VM), U2.2 (GND)
Other:
- moved on the sheet: C4, U1

Commit message: moved TP4057 closer to the VBAT
Parts:
- U3: footprint Package_TO_SOT_SMD:TSOT-23-6 -> SparkFun-Semiconductor-Standard:SOT23-6-Tight
Changed lines of the file:
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@@
 			)
 		)
-		(property "Footprint" "Package_TO_SOT_SMD:TSOT-23-6"
+		(property "Footprint" "SparkFun-Semiconductor-Standard:SOT23-6-Tight"
 			(at 102.87 85.09 0)
 			(effects

Commit message: v2.7 boxes
Parts:
- removed SW1: SW_DIP_x01, FlashlightLib:KCD11-2P, symbol Switch:SW_DIP_x01
- added U5: SS12J01_071, JLCPCB-SS12J01:SW-TH_SHOU-HAN_SS12J01, symbol SS12J01_071:SS12J01_071
Connections:
- net at D4.1 (K), Q2.2 (S): now also U5.2
- net at C3.1, L1.1, U2.4 (EN)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: now also U5.3
Changed lines of the file:
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@@
+	(wire
+		(pts
+			(xy 180.34 55.88) (xy 180.34 58.42)
+		)
+		(stroke
+			(width 0)
+			(type default)
+		)
+	)
 	(wire
 		(pts
@@
 	(wire
 		(pts
-			(xy 165.1 58.42) (xy 168.91 58.42)
+			(xy 165.1 58.42) (xy 177.8 58.42)
 		)
 		(stroke
@@
 	(wire
 		(pts
-			(xy 184.15 58.42) (xy 190.5 58.42)
+			(xy 177.8 58.42) (xy 177.8 55.88)
 		)
 		(stroke
@@
 		(pts
 			(xy 231.14 77.47) (xy 252.73 77.47)
+		)
+		(stroke
+			(width 0)
+			(type default)
+		)
+	)
+	(wire
+		(pts
+			(xy 180.34 58.42) (xy 190.5 58.42)
 		)
 		(stroke
@@
 				(justify left)
 				(hide yes)
-			)
-		)
-	)
-	(symbol
-		(lib_id "Switch:SW_DIP_x01")
-		(at 176.53 58.42 0)
-		(unit 1)
-		(exclude_from_sim no)
-		(in_bom no)
-		(on_board yes)
-		(dnp yes)
-		(fields_autoplaced yes)
-		(property "Reference" "SW1"
-			(at 176.53 50.8 0)
-			(effects
-				(font
-					(size 1.27 1.27)
-				)
-			)
-		)
-		(property "Value" "SW_DIP_x01"
-			(at 176.53 53.34 0)
-			(effects
-				(font
-					(size 1.27 1.27)
-				)
-			)
-		)
-		(property "Footprint" "FlashlightLib:KCD11-2P"
-			(at 176.53 58.42 0)
-			(effects
-				(font
-					(size 1.27 1.27)
-				)
-				(hide yes)
-			)
-		)
-		(property "Datasheet" "~"
-			(at 176.53 58.42 0)
-			(effects
-				(font
-					(size 1.27 1.27)
-				)
-				(hide yes)
-			)
-		)
-		(property "Description" "1x DIP Switch, Single Pole Single Throw (SPST) switch, small symbol"
-			(at 176.53 58.42 0)
-			(effects
-				(font
-					(size 1.27 1.27)
-				)
-				(hide yes)
-			)
-		)
-		(pin "1"
-		)
-		(pin "2"
-		)
-		(instances
-			(project "flashlight"
-				(path "/98487160-c149-430f-8381-4af03ebcbf31"
-					(reference "SW1")
-					(unit 1)
-				)
 			)
 		)
@@
 					(unit 1)
 				)
+			)
+		)
+	)
+	(symbol
+		(lib_id "SS12J01_071:SS12J01_071")
+		(at 177.8 53.34 0)
+		(unit 1)
+		(exclude_from_sim no)
+		(in_bom no)
+		(on_board yes)
+		(dnp yes)
+		(fields_autoplaced yes)
+		(property "Reference" "U5"
+			(at 181.61 49.9109 0)
+			(effects
+				(font
+					(size 1.27 1.27)
+				)
+				(justify left)
+			)
+		)
+		(property "Value" "SS12J01_071"
+			(at 181.61 52.4509 0)
+			(effects
+				(font
+					(size 1.27 1.27)
+				)
+				(justify left)
+			)
+		)
+		(property "Footprint" "JLCPCB-SS12J01:SW-TH_SHOU-HAN_SS12J01"
+			(at 177.8 63.5 0)
+			(effects
+				(font
+					(size 1.27 1.27)
+					(italic yes)
+				)
+				(hide yes)
+			)
+		)
+		(property "Datasheet" "https://atta.szlcsc.com/upload/public/pdf/source/20210820/C8D204FD916E0419E3F50724706D9DFB.pdf"
+			(at 175.514 53.213 0)
+			(effects
+				(font
+					(size 1.27 1.27)
+				)
+				(justify left)
+				(hide yes)
+			)
+		)
+		(property "Description" ""
+			(at 177.8 53.34 0)
+			(effects
+				(font
+					(size 1.27 1.27)
+				)
+				(hide yes)
+			)
+		)
+		(property "LCSC" "C2887258"
+			(at 177.8 53.34 0)
+			(effects
+				(font
+					(size 1.27 1.27)
+				)
+				(hide yes)
+			)
+		)
+		(pin "1"
+		)
+		(pin "2"
+		)
+		(pin "3"
+		)
+		(instances
+			(project "flashlight"
+				(path "/98487160-c149-430f-8381-4af03ebcbf31"
+					(reference "U5")
+					(unit 1)
+				)

Commit message: V3.0 21700 3x8 leds
Parts:
- removed J1: USB_B_Micro, FlashlightLib:USB-1101IPX6-02, symbol Connector:USB_B_Micro
- removed J2: Conn_01x03_Pin, FlashlightLib:LED_Strip, symbol Connector:Conn_01x03_Pin
- removed U3: TP4057, SparkFun-Semiconductor-Standard:SOT23-6-Tight, symbol Battery_Management:TP4057
- added C5, C6: 10uF/10V, Capacitor_SMD:C_0603_1608Metric, symbol Device:C
- added D10, D14, D15, D16, D18, D19, D21, D24, D26, D3, D7: LED, footprint:LED-SMD_L3.0-W1.4-RD_WHITE, symbol Device:LED
- added D11, D12, D13, D17, D20, D22, D23, D25, D27, D28, D6, D8, D9: LED_Pad, footprint:LED-SMD_3P-L5.7-W3.0-RD, symbol Device:LED_Pad
- added D2: D_Schottky, Diode_SMD:D_SMB, symbol Device:D_Schottky
- added F2: BSMD1210-150-6V, Fuse:Fuse_1210_3225Metric, symbol Device:Fuse
- added FB1: FerriteBead, Inductor_SMD:L_0805_2012Metric, symbol Device:FerriteBead
- added H1, H2, H3, H4: MountingHole, FlashlightLib:M4-insert, symbol Mechanical:MountingHole
- added J11: USB_C_Receptacle_USB2.0_16P, footprint:USB-SMD_GT-USB-7070A01, symbol ESP32S3LoRa:USB_C_Receptacle_USB2.0_16P
- added L2: 10uH, FlashlightLib:L_5.0x5.0, symbol Device:L
- added R20, R21: 5.1k, Resistor_SMD:R_0402_1005Metric, symbol Device:R
- added R5, R9: 33, Resistor_SMD:R_1206_3216Metric_Pad1.30x1.75mm_HandSolder, symbol Device:R
- added R8: 0.05, Resistor_SMD:R_1206_3216Metric, symbol Device:R
- added U3: TP5000, footprint:ESOP-8_L4.9-W3.9-P1.27-LS6.0-BL-EP, symbol MySymbols:TP5000
- BT1: footprint FlashlightLib:BH-18650_NoHole -> footprint:BAT-SMD_L82.5.5-W25-BH-21700-B1BJ001; LCSC C2988620 -> C20606791; now fitted; now in the parts list
- C1: value 22uF/25V -> 10uF/10V; footprint Capacitor_SMD:C_0805_2012Metric -> Capacitor_SMD:C_0603_1608Metric; LCSC C45783 -> C19702
- C3, C4: value 22uF/25V -> 22uF/35V; LCSC C45783 -> C6119901
- R1: value 1k -> 33; footprint Resistor_SMD:R_0603_1608Metric -> Resistor_SMD:R_1206_3216Metric_Pad1.30x1.75mm_HandSolder; LCSC C21190 -> C18005
- R6: value 10k -> 5.23k; footprint Resistor_SMD:R_0603_1608Metric -> Resistor_SMD:R_0805_2012Metric_Pad1.20x1.40mm_HandSolder; LCSC C25804 -> C2933464
- U1: footprint FlashlightLib:XB4908A -> footprint:ESN-4_L2.8-W2.3-LS3.7-BL
- U4: footprint MyFootprints:R6BHC-A05_LED -> footprint:LED-ARRAY-SMD_4P-L1.6-W1.3-BR-FD
- U5: footprint JLCPCB-SS12J01:SW-TH_SHOU-HAN_SS12J01 -> footprint:SW-TH_SHOU-HAN_SS12J01; now fitted; now in the parts list
Connections:
- net Earth_Protective: now also D11.1 (K), D11.3 (PAD), D12.3 (PAD), D13.3 (PAD), D17.3 (PAD), D19.1 (K), D20.1 (K), D20.3 (PAD), D22.3 (PAD), D23.3 (PAD), D25.3 (PAD), D27.3 (PAD), D28.3 (PAD), D6.3 (PAD), D8.3 (PAD), D9.3 (PAD)
- net GND: now also C5.2, C6.2, D2.2 (A), J11.A1 (GND), J11.A12 (GND), J11.B1 (GND), J11.B12 (GND), R20.2, R21.2, U3.2 (GND), U3.5 (TS), U3.9 (GND); no longer R1.2
- net VOUT: now also R1.2, R5.2, R9.2
- net at C1.1, D1.1 (K), D4.2 (A)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: now also U3.8 (VIN)
- net at BT1.1 (+), Q2.3 (D), R3.2: now also C6.1, R8.2, U3.4 (BAT)
- net at U4.2 (Blue-): now also U3.6 (~{STDBY})
- net at U4.4 (Red-): now also U3.7 (~{CHRG})
- net at C3.1, L1.1, U2.4 (EN)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: now also U5.1; no longer U5.3
- net at D1.2 (A): now also FB1.2
- net at R1.1: now also D27.2 (A)
- new net: D8.1 (K), D9.2 (A)
- new net: D7.1 (K), D8.2 (A)
- new net: D28.1 (K), D3.2 (A)
- new net: D28.2 (A), R9.1
- new net: D18.1 (K), D19.2 (A)
- new net: D17.1 (K), D18.2 (A)
- new net: D25.2 (A), D26.1 (K)
- new net: D26.2 (A), D27.1 (K)
- new net: D14.1 (K), D15.2 (A)
- new net: D13.1 (K), D14.2 (A)
- new net: D22.2 (A), D23.1 (K)
- new net: D23.2 (A), D24.1 (K)
- new net: D2.1 (K), L2.1, U3.1 (LX)
- new net: D6.1 (K), D7.2 (A)
- new net: D3.1 (K), D6.2 (A)
- new net: D24.2 (A), D25.1 (K)
- new net: C5.1, L2.2, R8.1, U3.3 (VS)
- new net: D10.1 (K), D11.2 (A)
- new net: D10.2 (A), D9.1 (K)
- new net: J11.A5 (CC1), R20.1
- new net: D16.1 (K), D17.2 (A)
- new net: D21.2 (A), D22.1 (K)
- new net: D15.1 (K), D16.2 (A)
- new net: D12.2 (A), R5.1
- new net: F2.1, J11.A4 (VBUS), J11.A9 (VBUS), J11.B4 (VBUS), J11.B9 (VBUS)
- new net: J11.B5 (CC2), R21.1
- new net: F2.2, FB1.1
- new net: D12.1 (K), D13.2 (A)
- new net: D20.2 (A), D21.1 (K)
- no-connect marks 4 -> 8
Other:
- note added: "23.5 V"
- note removed: "12.6V"
- moved on the sheet: C1, C2, C3, D1, D4, D5, L1, Q2, R2, R3, R4, R6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
